File: HardwareEngineering/lab/oneBitAdderCad/oneBitAdderCad.kicad_sch (KiCad schematic)
At the start: 0 parts

Commit message: Update oneBitAdderCad.kicad_sch
Other:
- title: (none) -> One Bit Adder
Changed lines of the file:
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@@
 (kicad_sch (version 20230121) (generator eeschema)
   (paper "A4")
+  (title_block
+    (title "One Bit Adder")
+    (date "2023-05-10")
+    (rev "1")
+  )
   (sheet_instances
     (path "/" (page "1"))

Commit message: update
Parts:
- added J2: Conn_01x03_Pin, symbol Connector:Conn_01x03_Pin
- added U1: 74HC86, symbol 74xx:74HC86
- added U2: 74LS32, symbol 74xx:74LS32
- added U3: 74LS08, symbol 74xx:74LS08
Connections:
- new net: J2.1 (Pin_1), U1.1, U3.1
- new net: J2.2 (Pin_2), U1.2, U3.2
- new net: U1.3, U1.4, U3.4
- new net: J2.3 (Pin_3), U1.5, U3.5
- new net: U2.1, U3.6
- new net: U2.2, U3.3

Commit message: Update
Parts:
- added J1: Conn_01x02_Socket, symbol Connector:Conn_01x02_Socket
Connections:
- net at U1.6: now also J1.1 (Pin_1)
- net at U2.3: now also J1.2 (Pin_2)
Changed lines of the file:
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@@
+    (stroke (width 0) (type default))
+  )
+  (wire (pts (xy 158.75 68.58) (xy 170.18 68.58))
     (stroke (width 0) (type default))
   )
@@
     (stroke (width 0) (type default))
   )
+  (wire (pts (xy 171.45 71.12) (xy 170.18 71.12))
+    (stroke (width 0) (type default))
+  )
   (wire (pts (xy 49.53 64.77) (xy 68.58 64.77))
     (stroke (width 0) (type default))
@@
     (stroke (width 0) (type default))
   )
+  (wire (pts (xy 158.75 71.12) (xy 158.75 68.58))
+    (stroke (width 0) (type default))
+  )
   (wire (pts (xy 68.58 64.77) (xy 71.12 64.77))
     (stroke (width 0) (type default))
@@
     (stroke (width 0) (type default))
   )
+  (wire (pts (xy 134.62 71.12) (xy 158.75 71.12))
+    (stroke (width 0) (type default))
+  )
   (wire (pts (xy 71.12 64.77) (xy 71.12 66.04))
+    (stroke (width 0) (type default))
+  )
+  (wire (pts (xy 171.45 85.09) (xy 171.45 71.12))
     (stroke (width 0) (type default))
   )
@@
     )
   )
+  (symbol (lib_id "Connector:Conn_01x02_Socket") (at 175.26 68.58 0) (unit 1)
+    (in_bom yes) (on_board yes) (dnp no) (fields_autoplaced)
+    (property "Reference" "J1" (at 176.53 69.215 0)
+      (effects (font (size 1.27 1.27)) (justify left))
+    )
+    (property "Value" "Conn_01x02_Socket" (at 176.53 71.755 0)
+      (effects (font (size 1.27 1.27)) (justify left))
+    )
+    (property "Footprint" "" (at 175.26 68.58 0)
+      (effects (font (size 1.27 1.27)) hide)
+    )
+    (property "Datasheet" "~" (at 175.26 68.58 0)
+      (effects (font (size 1.27 1.27)) hide)
+    )
+    (pin "1")
+    (pin "2")
+    (instances
+      (project "oneBitAdderCad"
+        (path "/dfa3bd34-6018-43f0-bf7d-75f255629607"
+          (reference "J1") (unit 1)
+        )
+      )
+    )
+  )
   (symbol (lib_id "Connector:Conn_01x03_Pin") (at 44.45 67.31 0) (unit 1)
     (in_bom yes) (on_board yes) (dnp no) (fields_autoplaced)
@@
     )
     (property "Footprint" "" (at 127 99.06 0)
-      (effects (font (size 1.27 1.27)) hide)
+      (effects (font (size 1.27 1.27)))
     )
     (property "Datasheet" "http://www.ti.com/lit/gpn/sn74LS08" (at 127 99.06 0)
